File: 555_PWM/555_PWM.sch (KiCad schematic (older format))
At the start: 1 part, among them U1 NE555

Commit message: накидал схему
Parts:
- added C1: 10uF, symbol Device:CP
- added C2: 0.1uF, symbol Device:C
- added R1, R5: 1K, Resistor_SMD:R_1206_3216Metric_Pad1.42x1.75mm_HandSolder, symbol Device:R
- added R2: 20K, Resistor_SMD:R_1206_3216Metric_Pad1.42x1.75mm_HandSolder, symbol Device:R
- added R3, R4: 2K, Resistor_SMD:R_1206_3216Metric_Pad1.42x1.75mm_HandSolder, symbol Device:R
- added R6: 50R, Resistor_SMD:R_1206_3216Metric_Pad1.42x1.75mm_HandSolder, symbol Device:R
- added RV1: R_POT, symbol Device:R_POT
- added U2: LM311, symbol Comparator:LM311
Connections:
- net +12V: now also U1.4 (R), R1.1, R3.1, R5.1, U2.8 (V+)
- net GND: now also C1.2, C2.2, R4.2, U2.1 (GND), U2.4 (V-)
- net at U1.2 (TR), U1.6 (THR): now also C2.1, R2.2, U2.3 (-)
- net at U1.5 (CV): now also C1.1
- net at U1.7 (DIS): now also R1.2, R2.1
- new net: RV1.2, U2.2 (+)
- new net: R5.2, R6.2, U2.7
- new net: R3.2, RV1.1
- new net: R4.1, RV1.3
Changed lines of the file:
@@
 	1    0    0    -1
 $EndComp
-Wire Wire Line
-	1850 3100 1850 2250
 $Comp
 L power:+12V #PWR?
@@
 $EndComp
 Wire Wire Line
-	1850 1450 1850 1000
+	1850 1450 1850 1300
 Wire Wire Line
 	1350 1650 1250 1650
@@
 Wire Wire Line
 	2450 2050 2350 2050
+Wire Wire Line
+	1350 2050 1150 2050
+Wire Wire Line
+	1150 2050 1150 1300
+Wire Wire Line
+	1150 1300 1850 1300
+Connection ~ 1850 1300
+Wire Wire Line
+	1850 1300 1850 1000
+$Comp
+L Device:CP C1
+U 1 1 5E57C679
+P 900 2050
+F 0 "C1" H 1018 2096 50  0000 L CNN
+F 1 "10uF" H 1018 2005 50  0000 L CNN
+F 2 "" H 938 1900 50  0001 C CNN
+F 3 "~" H 900 2050 50  0001 C CNN
+	1    900  2050
+	1    0    0    -1
+$EndComp
+Wire Wire Line
+	1350 1850 900  1850
+Wire Wire Line
+	900  1850 900  1900
+Wire Wire Line
+	900  2200 900  2500
+Wire Wire Line
+	900  2500 1850 2500
+Connection ~ 1850 2500
+Wire Wire Line
+	1850 2500 1850 2250
+$Comp
+L Device:R R2
+U 1 1 5E57D591
+P 2600 2050
+F 0 "R2" H 2670 2096 50  0000 L CNN
+F 1 "20K" H 2670 2005 50  0000 L CNN
+F 2 "Resistor_SMD:R_1206_3216Metric_Pad1.42x1.75mm_HandSolder" V 2530 2050 50  0001 C CNN
+F 3 "~" H 2600 2050 50  0001 C CNN
+	1    2600 2050
+	1    0    0    -1
+$EndComp
+Wire Wire Line
+	2600 2200 2600 2300
+Wire Wire Line
+	2600 2300 2450 2300
+Connection ~ 2450 2300
+Wire Wire Line
+	2350 1850 2600 1850
+Wire Wire Line
+	2600 1850 2600 1900
+$Comp
+L Device:R R1
+U 1 1 5E57E30E
+P 2600 1650
+F 0 "R1" H 2670 1696 50  0000 L CNN
+F 1 "1K" H 2670 1605 50  0000 L CNN
+F 2 "Resistor_SMD:R_1206_3216Metric_Pad1.42x1.75mm_HandSolder" V 2530 1650 50  0001 C CNN
+F 3 "~" H 2600 1650 50  0001 C CNN
+	1    2600 1650
+	1    0    0    -1
+$EndComp
+Wire Wire Line
+	2600 1800 2600 1850
+Connection ~ 2600 1850
+Wire Wire Line
+	2600 1500 2600 1300
+Wire Wire Line
+	2600 1300 1850 1300
+$Comp
+L Device:C C2
+U 1 1 5E57EF63
+P 2450 2550
+F 0 "C2" H 2565 2596 50  0000 L CNN
+F 1 "0.1uF" H 2565 2505 50  0000 L CNN
+F 2 "" H 2488 2400 50  0001 C CNN
+F 3 "~" H 2450 2550 50  0001 C CNN
+	1    2450 2550
+	1    0    0    -1
+$EndComp
+Wire Wire Line
+	2450 2400 2450 2300
+$Comp
+L Comparator:LM311 U2
+U 1 1 5E580ADE
+P 3750 1950
+F 0 "U2" H 3700 2350 50  0000 L CNN
+F 1 "LM311" H 3750 1800 50  0000 L CNN
+F 2 "" H 3750 1950 50  0001 C CNN
+F 3 "http://www.ti.com/lit/ds/symlink/lm311.pdf" H 3750 1950 50  0001 C CNN
+	1    3750 1950
+	1    0    0    -1
+$EndComp
+Wire Wire Line
+	1850 2500 1850 3050
+Wire Wire Line
+	2450 2700 2450 3050
+Wire Wire Line
+	2450 3050 1850 3050
+Connection ~ 1850 3050
+Wire Wire Line
+	1850 3050 1850 3100
+Wire Wire Line
+	3750 3050 3750 2300
+Connection ~ 2450 3050
+Wire Wire Line
+	3650 2250 3650 2300
+Wire Wire Line
+	3650 2300 3750 2300
+Connection ~ 3750 2300
+Wire Wire Line
+	3750 2300 3750 2250
+Wire Wire Line
+	3650 1650 3650 1300
+Connection ~ 2600 1300
+Wire Wire Line
+	2450 3050 3200 3050
+Wire Wire Line
+	2600 1300 3200 1300
+Wire Wire Line
+	2600 2300 3400 2300
+Wire Wire Line
+	3400 2300 3400 2050
+Wire Wire Line
+	3400 2050 3450 2050
+Connection ~ 2600 2300
+$Comp
+L Device:R_POT RV1
+U 1 1 5E585483
+P 3200 1850
+F 0 "RV1" H 3131 1896 50  0000 R CNN
+F 1 "R_POT" H 3131 1805 50  0000 R CNN
+F 2 "" H 3200 1850 50  0001 C CNN
+F 3 "~" H 3200 1850 50  0001 C CNN
+	1    3200 1850
+	1    0    0    -1
+$EndComp
+Wire Wire Line
+	3450 1850 3350 1850
+$Comp
+L Device:R R3
+U 1 1 5E5868AC
+P 3200 1500
+F 0 "R3" H 3270 1546 50  0000 L CNN
+F 1 "2K" H 3270 1455 50  0000 L CNN
+F 2 "Resistor_SMD:R_1206_3216Metric_Pad1.42x1.75mm_HandSolder" V 3130 1500 50  0001 C CNN
+F 3 "~" H 3200 1500 50  0001 C CNN
+	1    3200 1500
+	1    0    0    -1
+$EndComp
+Wire Wire Line
+	3200 1700 3200 1650
+Wire Wire Line
+	3200 1350 3200 1300
+Connection ~ 3200 1300
+Wire Wire Line
+	3200 1300 3650 1300
+$Comp
+L Device:R R4
+U 1 1 5E587C9E
+P 3200 2600
+F 0 "R4" H 3270 2646 50  0000 L CNN
+F 1 "2K" H 3270 2555 50  0000 L CNN
+F 2 "Resistor_SMD:R_1206_3216Metric_Pad1.42x1.75mm_HandSolder" V 3130 2600 50  0001 C CNN
+F 3 "~" H 3200 2600 50  0001 C CNN
+	1    3200 2600
+	1    0    0    -1
+$EndComp
+Wire Wire Line
+	3200 2000 3200 2450
+Wire Wire Line
+	3200 2750 3200 3050
+Connection ~ 3200 3050
+Wire Wire Line
+	3200 3050 3750 3050
+$Comp
+L Device:R R5
+U 1 1 5E588FC2
+P 4150 1600
+F 0 "R5" H 4220 1646 50  0000 L CNN
+F 1 "1K" H 4220 1555 50  0000 L CNN
+F 2 "Resistor_SMD:R_1206_3216Metric_Pad1.42x1.75mm_HandSolder" V 4080 1600 50  0001 C CNN
+F 3 "~" H 4150 1600 50  0001 C CNN
+	1    4150 1600
+	1    0    0    -1
+$EndComp
+Wire Wire Line
+	4150 1450 4150 1300
+Wire Wire Line
+	4150 1300 3650 1300
+Connection ~ 3650 1300
+Wire Wire Line
+	4050 1950 4150 1950
+Wire Wire Line
+	4150 1950 4150 1750
+$Comp
+L Device:R R6
+U 1 1 5E58A8F5
+P 4450 1950
+F 0 "R6" V 4243 1950 50  0000 C CNN
+F 1 "50R" V 4334 1950 50  0000 C CNN
+F 2 "Resistor_SMD:R_1206_3216Metric_Pad1.42x1.75mm_HandSolder" V 4380 1950 50  0001 C CNN
+F 3 "~" H 4450 1950 50  0001 C CNN
+	1    4450 1950
+	0    1    1    0
+$EndComp
+Wire Wire Line
+	4300 1950 4150 1950
+Connection ~ 4150 1950
 $EndSCHEMATC

Commit message: commit
Parts:
- added C3: 0.1uF, Capacitor_THT:C_Disc_D4.3mm_W1.9mm_P5.00mm, symbol Device:C
- C2: footprint (none) -> Capacitor_THT:C_Disc_D4.3mm_W1.9mm_P5.00mm
- RV1: footprint (none) -> Connector_PinHeader_2.54mm:PinHeader_1x03_P2.54mm_Vertical
- U2: footprint (none) -> Package_DIP:DIP-8_W7.62mm
Connections:
- net +12V: now also C3.2
- net GND: now also C3.1
Changed lines of the file:
@@
 F 0 "C2" H 2565 2596 50  0000 L CNN
 F 1 "0.1uF" H 2565 2505 50  0000 L CNN
-F 2 "" H 2488 2400 50  0001 C CNN
+F 2 "Capacitor_THT:C_Disc_D4.3mm_W1.9mm_P5.00mm" H 2488 2400 50  0001 C CNN
 F 3 "~" H 2450 2550 50  0001 C CNN
 	1    2450 2550
@@
 F 0 "U2" H 3700 2350 50  0000 L CNN
 F 1 "LM311" H 3750 1800 50  0000 L CNN
-F 2 "" H 3750 1950 50  0001 C CNN
+F 2 "Package_DIP:DIP-8_W7.62mm" H 3750 1950 50  0001 C CNN
 F 3 "http://www.ti.com/lit/ds/symlink/lm311.pdf" H 3750 1950 50  0001 C CNN
 	1    3750 1950
@@
 F 0 "RV1" H 3131 1896 50  0000 R CNN
 F 1 "R_POT" H 3131 1805 50  0000 R CNN
-F 2 "" H 3200 1850 50  0001 C CNN
+F 2 "Connector_PinHeader_2.54mm:PinHeader_1x03_P2.54mm_Vertical" H 3200 1850 50  0001 C CNN
 F 3 "~" H 3200 1850 50  0001 C CNN
 	1    3200 1850
@@
 	4300 1950 4150 1950
 Connection ~ 4150 1950
+$Comp
+L Device:C C3
+U 1 1 5E58D313
+P 3650 1100
+F 0 "C3" H 3765 1146 50  0000 L CNN
+F 1 "0.1uF" H 3765 1055 50  0000 L CNN
+F 2 "Capacitor_THT:C_Disc_D4.3mm_W1.9mm_P5.00mm" H 3688 950 50  0001 C CNN
+F 3 "~" H 3650 1100 50  0001 C CNN
+	1    3650 1100
+	1    0    0    -1
+$EndComp
+Wire Wire Line
+	3650 1250 3650 1300
+$Comp
+L power:GND #PWR?
+U 1 1 5E58F15E
+P 3350 950
+F 0 "#PWR?" H 3350 700 50  0001 C CNN
+F 1 "GND" H 3355 777 50  0000 C CNN
+F 2 "" H 3350 950 50  0001 C CNN
+F 3 "" H 3350 950 50  0001 C CNN
+	1    3350 950
+	1    0    0    -1
+$EndComp
+Wire Wire Line
+	3650 950  3650 900
+Wire Wire Line
+	3650 900  3350 900
+Wire Wire Line
+	3350 900  3350 950
 $EndSCHEMATC

Commit message: commit
Parts:
- added C4: 0.1uF, Capacitor_THT:C_Disc_D4.3mm_W1.9mm_P5.00mm, symbol Device:C
- added J1, J2: Screw_Terminal_01x02, TerminalBlock:TerminalBlock_bornier-2_P5.08mm, symbol Connector:Screw_Terminal_01x02
- added Q1: Q_PMOS_DGS, symbol Device:Q_PMOS_DGS
- R3, R4: value 2K -> 5K
Connections:
- net +12V: now also J2.1 (Pin_1), Q1.3 (S)
- net GND: now also C4.2, J1.2 (Pin_2), J2.2 (Pin_2)
- net at RV1.2, U2.2 (+): now also C4.1
- net at R6.1: now also Q1.2 (G)
- new net: J1.1 (Pin_1), Q1.1 (D)
Other:
- moved on the sheet: C3, R5, R6, U2
Changed lines of the file:
@@
 L Comparator:LM311 U2
 U 1 1 5E580ADE
-P 3750 1950
-F 0 "U2" H 3700 2350 50  0000 L CNN
-F 1 "LM311" H 3750 1800 50  0000 L CNN
-F 2 "Package_DIP:DIP-8_W7.62mm" H 3750 1950 50  0001 C CNN
-F 3 "http://www.ti.com/lit/ds/symlink/lm311.pdf" H 3750 1950 50  0001 C CNN
-	1    3750 1950
+P 3950 1950
+F 0 "U2" H 3900 2350 50  0000 L CNN
+F 1 "LM311" H 3950 1800 50  0000 L CNN
+F 2 "Package_DIP:DIP-8_W7.62mm" H 3950 1950 50  0001 C CNN
+F 3 "http://www.ti.com/lit/ds/symlink/lm311.pdf" H 3950 1950 50  0001 C CNN
+	1    3950 1950
 	1    0    0    -1
 $EndComp
@@
 	1850 3050 1850 3100
 Wire Wire Line
-	3750 3050 3750 2300
+	3950 3050 3950 2300
 Connection ~ 2450 3050
 Wire Wire Line
-	3650 2250 3650 2300
-Wire Wire Line
-	3650 2300 3750 2300
-Connection ~ 3750 2300
-Wire Wire Line
-	3750 2300 3750 2250
-Wire Wire Line
-	3650 1650 3650 1300
+	3850 2250 3850 2300
+Wire Wire Line
+	3850 2300 3950 2300
+Connection ~ 3950 2300
+Wire Wire Line
+	3950 2300 3950 2250
+Wire Wire Line
+	3850 1650 3850 1300
 Connection ~ 2600 1300
 Wire Wire Line
@@
 	2600 1300 3200 1300
 Wire Wire Line
-	2600 2300 3400 2300
-Wire Wire Line
-	3400 2300 3400 2050
-Wire Wire Line
-	3400 2050 3450 2050
-Connection ~ 2600 2300
+	2600 2300 2900 2300
+Wire Wire Line
+	2900 2300 2900 2050
+Wire Wire Line
+	2900 2050 3650 2050
 $Comp
 L Device:R_POT RV1
@@
 $EndComp
 Wire Wire Line
-	3450 1850 3350 1850
+	3650 1850 3450 1850
 $Comp
 L Device:R R3
@@
 P 3200 1500
 F 0 "R3" H 3270 1546 50  0000 L CNN
-F 1 "2K" H 3270 1455 50  0000 L CNN
+F 1 "5K" H 3270 1455 50  0000 L CNN
 F 2 "Resistor_SMD:R_1206_3216Metric_Pad1.42x1.75mm_HandSolder" V 3130 1500 50  0001 C CNN
 F 3 "~" H 3200 1500 50  0001 C CNN
@@
 Wire Wire Line
 	3200 1350 3200 1300
-Connection ~ 3200 1300
-Wire Wire Line
-	3200 1300 3650 1300
+Wire Wire Line
+	3200 1300 3850 1300
 $Comp
 L Device:R R4
@@
 P 3200 2600
 F 0 "R4" H 3270 2646 50  0000 L CNN
-F 1 "2K" H 3270 2555 50  0000 L CNN
+F 1 "5K" H 3270 2555 50  0000 L CNN
 F 2 "Resistor_SMD:R_1206_3216Metric_Pad1.42x1.75mm_HandSolder" V 3130 2600 50  0001 C CNN
 F 3 "~" H 3200 2600 50  0001 C CNN
@@
 Wire Wire Line
 	3200 2750 3200 3050
-Connection ~ 3200 3050
-Wire Wire Line
-	3200 3050 3750 3050
+Wire Wire Line
+	3200 3050 3450 3050
 $Comp
 L Device:R R5
 U 1 1 5E588FC2
-P 4150 1600
-F 0 "R5" H 4220 1646 50  0000 L CNN
-F 1 "1K" H 4220 1555 50  0000 L CNN
-F 2 "Resistor_SMD:R_1206_3216Metric_Pad1.42x1.75mm_HandSolder" V 4080 1600 50  0001 C CNN
-F 3 "~" H 4150 1600 50  0001 C CNN
-	1    4150 1600
-	1    0    0    -1
-$EndComp
-Wire Wire Line
-	4150 1450 4150 1300
-Wire Wire Line
-	4150 1300 3650 1300
-Connection ~ 3650 1300
-Wire Wire Line
-	4050 1950 4150 1950
-Wire Wire Line
-	4150 1950 4150 1750
+P 4350 1600
+F 0 "R5" H 4420 1646 50  0000 L CNN
+F 1 "1K" H 4420 1555 50  0000 L CNN
+F 2 "Resistor_SMD:R_1206_3216Metric_Pad1.42x1.75mm_HandSolder" V 4280 1600 50  0001 C CNN
+F 3 "~" H 4350 1600 50  0001 C CNN
+	1    4350 1600
+	1    0    0    -1
+$EndComp
+Wire Wire Line
+	4350 1450 4350 1300
+Wire Wire Line
+	4350 1300 3850 1300
+Connection ~ 3850 1300
+Wire Wire Line
+	4250 1950 4350 1950
+Wire Wire Line
+	4350 1950 4350 1750
 $Comp
 L Device:R R6
 U 1 1 5E58A8F5
-P 4450 1950
-F 0 "R6" V 4243 1950 50  0000 C CNN
-F 1 "50R" V 4334 1950 50  0000 C CNN
-F 2 "Resistor_SMD:R_1206_3216Metric_Pad1.42x1.75mm_HandSolder" V 4380 1950 50  0001 C CNN
-F 3 "~" H 4450 1950 50  0001 C CNN
-	1    4450 1950
+P 4650 1950
+F 0 "R6" V 4443 1950 50  0000 C CNN
+F 1 "50R" V 4534 1950 50  0000 C CNN
+F 2 "Resistor_SMD:R_1206_3216Metric_Pad1.42x1.75mm_HandSolder" V 4580 1950 50  0001 C CNN
+F 3 "~" H 4650 1950 50  0001 C CNN
+	1    4650 1950
 	0    1    1    0
 $EndComp
 Wire Wire Line
-	4300 1950 4150 1950
-Connection ~ 4150 1950
+	4500 1950 4350 1950
+Connection ~ 4350 1950
 $Comp
 L Device:C C3
 U 1 1 5E58D313
-P 3650 1100
-F 0 "C3" H 3765 1146 50  0000 L CNN
-F 1 "0.1uF" H 3765 1055 50  0000 L CNN
-F 2 "Capacitor_THT:C_Disc_D4.3mm_W1.9mm_P5.00mm" H 3688 950 50  0001 C CNN
-F 3 "~" H 3650 1100 50  0001 C CNN
-	1    3650 1100
-	1    0    0    -1
-$EndComp
-Wire Wire Line
-	3650 1250 3650 1300
+P 3850 1100
+F 0 "C3" H 3965 1146 50  0000 L CNN
+F 1 "0.1uF" H 3965 1055 50  0000 L CNN
+F 2 "Capacitor_THT:C_Disc_D4.3mm_W1.9mm_P5.00mm" H 3888 950 50  0001 C CNN
+F 3 "~" H 3850 1100 50  0001 C CNN
+	1    3850 1100
+	1    0    0    -1
+$EndComp
+Wire Wire Line
+	3850 1250 3850 1300
 $Comp
 L power:GND #PWR?
 U 1 1 5E58F15E
-P 3350 950
-F 0 "#PWR?" H 3350 700 50  0001 C CNN
-F 1 "GND" H 3355 777 50  0000 C CNN
-F 2 "" H 3350 950 50  0001 C CNN
-F 3 "" H 3350 950 50  0001 C CNN
-	1    3350 950
-	1    0    0    -1
-$EndComp
-Wire Wire Line
-	3650 950  3650 900
-Wire Wire Line
-	3650 900  3350 900
-Wire Wire Line
-	3350 900  3350 950
+P 3550 950
+F 0 "#PWR?" H 3550 700 50  0001 C CNN
+F 1 "GND" H 3555 777 50  0000 C CNN
+F 2 "" H 3550 950 50  0001 C CNN
+F 3 "" H 3550 950 50  0001 C CNN
+	1    3550 950
+	1    0    0    -1
+$EndComp
+Wire Wire Line
+	3850 950  3850 900
+Wire Wire Line
+	3850 900  3550 900
+Wire Wire Line
+	3550 900  3550 950
+$Comp
+L Device:Q_PMOS_DGS Q1
+U 1 1 5E590E7D
+P 5100 1950
+F 0 "Q1" H 5000 1800 50  0000 L CNN
+F 1 "Q_PMOS_DGS" H 4650 2150 50  0000 L CNN
+F 2 "" H 5300 2050 50  0001 C CNN
+F 3 "~" H 5100 1950 50  0001 C CNN
+	1    5100 1950
+	1    0    0    1
+$EndComp
+Wire Wire Line
+	5200 1750 5200 1300
+Wire Wire Line
+	5200 1300 4350 1300
+Connection ~ 4350 1300
+Wire Wire Line
+	4900 1950 4800 1950
+$Comp
+L Connector:Screw_Terminal_01x02 J1
+U 1 1 5E59584B
+P 5650 2300
+F 0 "J1" H 5730 2292 50  0000 L CNN
+F 1 "Screw_Terminal_01x02" H 5730 2201 50  0000 L CNN
+F 2 "TerminalBlock:TerminalBlock_bornier-2_P5.08mm" H 5650 2300 50  0001 C CNN
+F 3 "~" H 5650 2300 50  0001 C CNN
+	1    5650 2300
+	1    0    0    -1
+$EndComp
+Wire Wire Line
+	5450 2300 5200 2300
+Wire Wire Line
+	5200 2300 5200 2150
+Wire Wire Line
+	5450 2400 5200 2400
+Wire Wire Line
+	5200 2400 5200 3050
+Wire Wire Line
+	5200 3050 3950 3050
+Connection ~ 3950 3050
+$Comp
+L Connector:Screw_Terminal_01x02 J2
+U 1 1 5E5983F3
+P 1250 4000
+F 0 "J2" H 1330 3992 50  0000 L CNN
+F 1 "Screw_Terminal_01x02" H 1330 3901 50  0000 L CNN
+F 2 "TerminalBlock:TerminalBlock_bornier-2_P5.08mm" H 1250 4000 50  0001 C CNN
+F 3 "~" H 1250 4000 50  0001 C CNN
+	1    1250 4000
+	1    0    0    -1
+$EndComp
+$Comp
+L power:GND #PWR?
+U 1 1 5E598CE9
+P 950 4200
+F 0 "#PWR?" H 950 3950 50  0001 C CNN
+F 1 "GND" H 955 4027 50  0000 C CNN
+F 2 "" H 950 4200 50  0001 C CNN
+F 3 "" H 950 4200 50  0001 C CNN
+	1    950  4200
+	1    0    0    -1
+$EndComp
+Wire Wire Line
+	1050 4100 950  4100
+Wire Wire Line
+	950  4100 950  4200
+$Comp
+L power:+12V #PWR?
+U 1 1 5E59A37B
+P 950 3900
+F 0 "#PWR?" H 950 3750 50  0001 C CNN
+F 1 "+12V" H 965 4073 50  0000 C CNN
+F 2 "" H 950 3900 50  0001 C CNN
+F 3 "" H 950 3900 50  0001 C CNN
+	1    950  3900
+	1    0    0    -1
+$EndComp
+Wire Wire Line
+	1050 4000 950  4000
+Wire Wire Line
+	950  4000 950  3900
+Connection ~ 3200 1300
+Connection ~ 3200 3050
+Connection ~ 2600 2300
+$Comp
+L Device:C C4
+U 1 1 5E5A7FEA
+P 3450 2300
+F 0 "C4" H 3565 2346 50  0000 L CNN
+F 1 "0.1uF" H 3565 2255 50  0000 L CNN
+F 2 "Capacitor_THT:C_Disc_D4.3mm_W1.9mm_P5.00mm" H 3488 2150 50  0001 C CNN
+F 3 "~" H 3450 2300 50  0001 C CNN
+	1    3450 2300
+	1    0    0    -1
+$EndComp
+Wire Wire Line
+	3450 2150 3450 1850
+Connection ~ 3450 1850
+Wire Wire Line
+	3450 1850 3350 1850
+Wire Wire Line
+	3450 2450 3450 3050
+Connection ~ 3450 3050
+Wire Wire Line
+	3450 3050 3950 3050
 $EndSCHEMATC

Commit message: начал трассировку
Parts:
- removed Q1: Q_PMOS_DGS, symbol Device:Q_PMOS_DGS
- added C6: 1000uF, Capacitor_THT:CP_Radial_D10.0mm_P5.00mm, symbol Device:CP
- added D1: 1N4148, Diode_THT:D_DO-35_SOD27_P10.16mm_Horizontal, symbol Diode:1N4148
- added Q1: Q_PMOS_GDS, Package_TO_SOT_THT:TO-220-3_Vertical, symbol Device:Q_PMOS_GDS
- C1: footprint (none) -> Capacitor_THT:CP_Radial_D5.0mm_P2.50mm
Connections:
- net +12V: now also C6.1, D1.1 (K), Q1.3 (S)
- net GND: now also C6.2
- net at R6.1: now also Q1.1 (G)
- net at J1.1 (Pin_1): now also D1.2 (A), Q1.2 (D)
Other:
- moved on the sheet: J2
Changed lines of the file:
@@
 $EndComp
 $Comp
-L power:GND #PWR?
+L power:GND #PWR0101
 U 1 1 5E57A19D
 P 1850 3100
-F 0 "#PWR?" H 1850 2850 50  0001 C CNN
+F 0 "#PWR0101" H 1850 2850 50  0001 C CNN
 F 1 "GND" H 1855 2927 50  0000 C CNN
 F 2 "" H 1850 3100 50  0001 C CNN
@@
 $EndComp
 $Comp
-L power:+12V #PWR?
+L power:+12V #PWR0102
 U 1 1 5E57ABC4
 P 1850 1000
-F 0 "#PWR?" H 1850 850 50  0001 C CNN
+F 0 "#PWR0102" H 1850 850 50  0001 C CNN
 F 1 "+12V" H 1865 1173 50  0000 C CNN
 F 2 "" H 1850 1000 50  0001 C CNN
@@
 F 0 "C1" H 1018 2096 50  0000 L CNN
 F 1 "10uF" H 1018 2005 50  0000 L CNN
-F 2 "" H 938 1900 50  0001 C CNN
+F 2 "Capacitor_THT:CP_Radial_D5.0mm_P2.50mm" H 938 1900 50  0001 C CNN
 F 3 "~" H 900 2050 50  0001 C CNN
 	1    900  2050
@@
 	3850 1250 3850 1300
 $Comp
-L power:GND #PWR?
+L power:GND #PWR0103
 U 1 1 5E58F15E
 P 3550 950
-F 0 "#PWR?" H 3550 700 50  0001 C CNN
+F 0 "#PWR0103" H 3550 700 50  0001 C CNN
 F 1 "GND" H 3555 777 50  0000 C CNN
 F 2 "" H 3550 950 50  0001 C CNN
@@
 Wire Wire Line
 	3550 900  3550 950
-$Comp
-L Device:Q_PMOS_DGS Q1
-U 1 1 5E590E7D
-P 5100 1950
-F 0 "Q1" H 5000 1800 50  0000 L CNN
-F 1 "Q_PMOS_DGS" H 4650 2150 50  0000 L CNN
-F 2 "" H 5300 2050 50  0001 C CNN
-F 3 "~" H 5100 1950 50  0001 C CNN
-	1    5100 1950
-	1    0    0    1
-$EndComp
-Wire Wire Line
-	5200 1750 5200 1300
+Wire Wire Line
+	5200 1750 5200 1700
 Wire Wire Line
 	5200 1300 4350 1300
@@
 	5450 2300 5200 2300
 Wire Wire Line
-	5200 2300 5200 2150
+	5200 2300 5200 2200
 Wire Wire Line
 	5450 2400 5200 2400
@@
 L Connector:Screw_Terminal_01x02 J2
 U 1 1 5E5983F3
-P 1250 4000
-F 0 "J2" H 1330 3992 50  0000 L CNN
-F 1 "Screw_Terminal_01x02" H 1330 3901 50  0000 L CNN
-F 2 "TerminalBlock:TerminalBlock_bornier-2_P5.08mm" H 1250 4000 50  0001 C CNN
-F 3 "~" H 1250 4000 50  0001 C CNN
-	1    1250 4000
-	1    0    0    -1
-$EndComp
-$Comp
-L power:GND #PWR?
+P 1300 3850
+F 0 "J2" H 1380 3842 50  0000 L CNN
+F 1 "Screw_Terminal_01x02" H 1380 3751 50  0000 L CNN
+F 2 "TerminalBlock:TerminalBlock_bornier-2_P5.08mm" H 1300 3850 50  0001 C CNN
+F 3 "~" H 1300 3850 50  0001 C CNN
+	1    1300 3850
+	1    0    0    -1
+$EndComp
+$Comp
+L power:GND #PWR0104
 U 1 1 5E598CE9
-P 950 4200
-F 0 "#PWR?" H 950 3950 50  0001 C CNN
-F 1 "GND" H 955 4027 50  0000 C CNN
-F 2 "" H 950 4200 50  0001 C CNN
-F 3 "" H 950 4200 50  0001 C CNN
-	1    950  4200
-	1    0    0    -1
-$EndComp
-Wire Wire Line
-	1050 4100 950  4100
-Wire Wire Line
-	950  4100 950  4200
-$Comp
-L power:+12V #PWR?
+P 1000 4050
+F 0 "#PWR0104" H 1000 3800 50  0001 C CNN
+F 1 "GND" H 1005 3877 50  0000 C CNN
+F 2 "" H 1000 4050 50  0001 C CNN
+F 3 "" H 1000 4050 50  0001 C CNN
+	1    1000 4050
+	1    0    0    -1
+$EndComp
+Wire Wire Line
+	1100 3950 1000 3950
+Wire Wire Line
+	1000 3950 1000 4050
+$Comp
+L power:+12V #PWR0105
 U 1 1 5E59A37B
-P 950 3900
-F 0 "#PWR?" H 950 3750 50  0001 C CNN
-F 1 "+12V" H 965 4073 50  0000 C CNN
-F 2 "" H 950 3900 50  0001 C CNN
-F 3 "" H 950 3900 50  0001 C CNN
-	1    950  3900
-	1    0    0    -1
-$EndComp
-Wire Wire Line
-	1050 4000 950  4000
-Wire Wire Line
-	950  4000 950  3900
+P 1000 3750
+F 0 "#PWR0105" H 1000 3600 50  0001 C CNN
+F 1 "+12V" H 1015 3923 50  0000 C CNN
+F 2 "" H 1000 3750 50  0001 C CNN
+F 3 "" H 1000 3750 50  0001 C CNN
+	1    1000 3750
+	1    0    0    -1
+$EndComp
+Wire Wire Line
+	1100 3850 1000 3850
+Wire Wire Line
+	1000 3850 1000 3750
 Connection ~ 3200 1300
 Connection ~ 3200 3050
@@
 Wire Wire Line
 	3450 3050 3950 3050
+$Comp
+L Device:Q_PMOS_GDS Q1
+U 1 1 5E5ABAA4
+P 5100 1950
+F 0 "Q1" H 4950 1850 50  0000 L CNN
+F 1 "Q_PMOS_GDS" H 4650 2100 50  0000 L CNN
+F 2 "Package_TO_SOT_THT:TO-220-3_Vertical" H 5300 2050 50  0001 C CNN
+F 3 "~" H 5100 1950 50  0001 C CNN
+	1    5100 1950
+	1    0    0    1
+$EndComp
+$Comp
+L Diode:1N4148 D1
+U 1 1 5E5AFFA2
+P 5400 1950
+F 0 "D1" V 5354 2029 50  0000 L CNN
+F 1 "1N4148" V 5445 2029 50  0000 L CNN
+F 2 "Diode_THT:D_DO-35_SOD27_P10.16mm_Horizontal" H 5400 1775 50  0001 C CNN
+F 3 "https://assets.nexperia.com/documents/data-sheet/1N4148_1N4448.pdf" H 5400 1950 50  0001 C CNN
+	1    5400 1950
+	0    1    1    0
+$EndComp
+Wire Wire Line
+	5400 2100 5400 2200
+Wire Wire Line
+	5400 2200 5200 2200
+Connection ~ 5200 2200
+Wire Wire Line
+	5200 2200 5200 2150
+Wire Wire Line
+	5400 1800 5400 1700
+Wire Wire Line
+	5400 1700 5200 1700
+Connection ~ 5200 1700
+Wire Wire Line
+	5200 1700 5200 1300
+$Comp
+L power:GND #PWR?
+U 1 1 5E5B9808
+P 2550 4200
+F 0 "#PWR?" H 2550 3950 50  0001 C CNN
+F 1 "GND" H 2555 4027 50  0000 C CNN
+F 2 "" H 2550 4200 50  0001 C CNN
+F 3 "" H 2550 4200 50  0001 C CNN
+	1    2550 4200
+	1    0    0    -1
+$EndComp
+Wire Wire Line
+	2550 4100 2550 4200
+$Comp
+L power:+12V #PWR?
+U 1 1 5E5B9810
+P 2550 3700
+F 0 "#PWR?" H 2550 3550 50  0001 C CNN
+F 1 "+12V" H 2565 3873 50  0000 C CNN
+F 2 "" H 2550 3700 50  0001 C CNN
+F 3 "" H 2550 3700 50  0001 C CNN
+	1    2550 3700
+	1    0    0    -1
+$EndComp
+Wire Wire Line
+	2550 3800 2550 3700
+$Comp
+L Device:CP C6
+U 1 1 5E5BC680
+P 2550 3950
+F 0 "C6" H 2668 3996 50  0000 L CNN
+F 1 "1000uF" H 2668 3905 50  0000 L CNN
+F 2 "Capacitor_THT:CP_Radial_D10.0mm_P5.00mm" H 2588 3800 50  0001 C CNN
+F 3 "~" H 2550 3950 50  0001 C CNN
+	1    2550 3950
+	1    0    0    -1
+$EndComp
 $EndSCHEMATC
